Commit message: Robot test env introduced.

File: lumi_description/robots/robot.urdf.xacro (robot description, xacro)
@@ -6,5 +6,5 @@
         <compiler meshdir="../meshes/" balanceinertia="true"/>
     </mujoco>
-    <link name="base_link"/>
+    <link name="base_link" />
     <xacro:panda_arm connected_to="base_link" arm_id="lumi"/>
     <xacro:hand ns="lumi" rpy="0 0 ${-pi/4}" connected_to="lumi_link8"/>

Commit message: hack fix gripper controller

File: lumi_description/robots/robot.urdf.xacro (robot description, xacro)
@@ -9,3 +9,9 @@
     <xacro:panda_arm connected_to="base_link" arm_id="lumi"/>
     <xacro:hand ns="lumi" rpy="0 0 ${-pi/4}" connected_to="lumi_link8"/>
+    <link name="lumi_ee"/>
+    <joint name="ee_fjoint" type="fixed">
+        <origin xyz="0 0 ${0.058 * 2}" rpy="0 0 0"/>
+        <parent link="lumi_hand"/>
+        <child link="lumi_ee"/>
+    </joint>
 </robot>

File: lumi_description/robots/robot_table_env.urdf.xacro (robot description, xacro)
@@ -22,3 +22,10 @@
     <xacro:panda_arm connected_to="base_link" arm_id="lumi" xyz="0 0 0"/>
     <xacro:hand ns="lumi" rpy="0 0 ${-pi/4}" connected_to="lumi_link8"/>
+    <!-- from master -->
+    <link name="lumi_ee"/>
+    <joint name="ee_fjoint" type="fixed">
+        <origin xyz="0 0 ${0.058 * 2}" rpy="0 0 0"/>
+        <parent link="lumi_hand"/>
+        <child link="lumi_ee"/>
+    </joint>
 </robot>
